File: Section B - MCU_sch.kicad_sch (KiCad schematic)
At the start: 10 parts, among them J2 USB_C_Receptacle_USB2.0_14P, SW2 TACTILE SWITCH, SW3 TACTILE SWITCH, U3 ESP32-S3-WROOM-1, U4 PESD2ETH-AXR_C5310973

Commit message: add CAN port, change power regulation
Parts:
- added C26, C27: 100nF, symbol Device:C
- added D1: PESD1CAN,215, easyeda2kicad:SOT-23_L2.9-W1.3-P1.90-LS2.4-BR, symbol easyeda2kicad:PESD1CAN,215
- added D2: LED_RGAB, symbol Device:LED_RGAB
- added J3: Conn_01x02_Pin, symbol Connector:Conn_01x02_Pin
- added R19: 120R, symbol Device:R
- added R22, R23: 5.1K, symbol Device:R
- added R24, R25, R26: 1K, symbol Device:R
- added U24: MCP2562-E-SN, Package_SO:SOIC-8_3.9x4.9mm_P1.27mm, symbol Interface_CAN_LIN:MCP2562-E-SN
- C10: value C -> 1uF
- C11: value C -> 10uF 10V
- C8: value C -> 100nF
- C9: value C -> 10uF
- R2: value R -> 10K
Connections:
- net +3.3V: now also C27.1, D2.3 (A), U24.5 (Vio)
- net +5V: now also C26.1, U24.3 (VDD)
- net GND: now also C26.2, C27.2, D1.3, R22.2, R23.2, U24.2 (VSS), U24.8 (STBY)
- net at J2.A5 (CC1): now also R22.1
- net at J2.B5 (CC2): now also R23.1
- new net: D1.1, J3.1 (Pin_1), U24.7 (CANH)
- new net: J3.2 (Pin_2), R19.1
- new net: D2.1 (RK), R24.2
- new net: D2.2 (GK), R25.2
- new net: D2.4 (BK), R26.2
- new net: D1.2, R19.2, U24.6 (CANL)
Other:
- moved on the sheet: C10, C11, C8, C9, J2, R2, SW2, SW3, U3, U4
